Commit message: troubleshooting

File: src/my_robot/urdf/my_robot.xacro (robot description, xacro)
@@ -156,4 +156,11 @@
       <dynamics damping="1.0" friction="1.0"/>
     </joint>
+  <joint name="camera_optical_joint" type="fixed">
+    <origin xyz="0 0 0" rpy="-1.5707 0 -1.5707"/>
+    <parent link="camera"/>
+    <child link="camera_link_optical"/>
+  </joint>
+  <link name="camera_link_optical">
+  </link>
 <link name='hokuyo'>
     <inertial>

Commit message: Updated plugin and xarco files

File: src/my_robot/urdf/my_robot.xacro (robot description, xacro)
@@ -59,5 +59,5 @@
     <inertial>
       <mass value="5.0"/>
-      <origin xyz="0.0 0 0" rpy="0 1.5707 1.5707"/>
+      <origin xyz="0.0 0 0" rpy="0 0 0"/>
       <inertia
           ixx="0.1" ixy="0" ixz="0"
@@ -82,5 +82,5 @@
     <inertial>
       <mass value="5.0"/>
-      <origin xyz="0.0 0 0" rpy="0 1.5707 1.5707"/>
+      <origin xyz="0.0 0 0" rpy="0 0 0"/>
       <inertia
           ixx="0.1" ixy="0" ixz="0"
@@ -148,4 +148,7 @@
     </visual>
 </link>
+<gazebo reference="camera">
+    <material>Gazebo/Black</material>
+</gazebo>
 <joint name="camera_joint" type="fixed">
       <origin xyz="0.2 0 0" rpy="0 0 0"/>
@@ -157,5 +160,5 @@
     </joint>
   <joint name="camera_optical_joint" type="fixed">
-    <origin xyz="0 0 0" rpy="-1.5707 0 -1.5707"/>
+    <origin xyz="0 0 0" rpy=" -1.5707 0 -1.5707"/>
     <parent link="camera"/>
     <child link="camera_link_optical"/>
@@ -185,5 +188,5 @@
 </link>
 <joint name="hokuyo_joint" type="fixed">
-      <origin xyz="0.15 0 0.1" rpy="0 0 0"/>
+      <origin xyz="0.15 0 0.08" rpy="0 0 0"/>
       <child link="hokuyo"/>
       <parent link="chassis"/>
